File: Arduino_Mega2560_Practice/Section_01_USB_ATmega16U2.kicad_sch (KiCad schematic)
At the start: 0 parts

Commit message: 4654156
Parts:
- added J1: USB_C_Receptacle_USB2.0_16P, Connector_USB:USB_C_Receptacle_GCT_USB4105-xx-A_16P_TopMnt_Horizontal, symbol Arduino_Mega2560_Lib:USB_C_16P
Connections:
- new net: J1.A1 (GND), J1.A12 (GND), J1.B1 (GND), J1.B12 (GND)
- new net: J1.A4 (VBUS), J1.A9 (VBUS), J1.B4 (VBUS), J1.B9 (VBUS)
Changed lines of the file:
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@@
 (kicad_sch
-	(version 20231120)
-	(generator "kicad_symbol_editor")
-	(generator_version "9.0")
+	(version 20260306)
+	(generator "eeschema")
+	(generator_version "10.0")
 	(paper "A4")
 	(title_block
@@
 		(comment 3 "Use symbols from: Arduino_Mega2560_Lib")
 	)
+	(symbol
+		(lib_id "Arduino_Mega2560_Lib:USB_C_16P")
+		(at 46.99 52.07 0)
+		(unit 1)
+		(body_style 1)
+		(exclude_from_sim no)
+		(in_bom yes)
+		(on_board yes)
+		(in_pos_files yes)
+		(dnp no)
+		(fields_autoplaced yes)
+		(property "Reference" "J1"
+			(at 46.99 29.21 0)
+			(show_name no)
+			(do_not_autoplace no)
+			(effects
+				(font
+					(size 1.27 1.27)
+				)
+			)
+		)
+		(property "Value" "USB_C_Receptacle_USB2.0_16P"
+			(at 46.99 31.75 0)
+			(show_name no)
+			(do_not_autoplace no)
+			(effects
+				(font
+					(size 1.27 1.27)
+				)
+			)
+		)
+		(property "Footprint" "Connector_USB:USB_C_Receptacle_GCT_USB4105-xx-A_16P_TopMnt_Horizontal"
+			(at 50.8 52.07 0)
+			(hide yes)
+			(show_name no)
+			(do_not_autoplace no)
+			(effects
+				(font
+					(size 1.27 1.27)
+				)
+			)
+		)
+		(property "Datasheet" "https://www.usb.org/sites/default/files/documents/usb_type-c.zip"
+			(at 50.8 52.07 0)
+			(hide yes)
+			(show_name no)
+			(do_not_autoplace no)
+			(effects
+				(font
+					(size 1.27 1.27)
+				)
+			)
+		)
+		(property "Description" "USB 2.0-only 16P Type-C Receptacle connector"
+			(at 46.99 52.07 0)
+			(hide yes)
+			(show_name no)
+			(do_not_autoplace no)
+			(effects
+				(font
+					(size 1.27 1.27)
+				)
+			)
+		)
+		(pin "A8"
+		)
+		(pin "B1"
+		)
+		(pin "A4"
+		)
+		(pin "A6"
+		)
+		(pin "B7"
+		)
+		(pin "B12"
+		)
+		(pin "A5"
+		)
+		(pin "A12"
+		)
+		(pin "A9"
+		)
+		(pin "B6"
+		)
+		(pin "B8"
+		)
+		(pin "B5"
+		)
+		(pin "B9"
+		)
+		(pin "S1"
+		)
+		(pin "A7"
+		)
+		(pin "B4"
+		)
+		(pin "A1"
+		)
+		(instances
+			(project "Arduino_Mega2560_Practice"
+				(path "/a1b2c3d4-0001-0000-0000-000000000001/a1b2c3d4-0001-0000-0000-000000000002"
+					(reference "J1")
+					(unit 1)
+				)
+			)
+		)
+	)
 	(sheet_instances
 		(path "/"
@@
 		)
 	)
+	(embedded_fonts no)
 )
